File: projects/FSAE/TeensyBalanceBoard2.1.sch (EAGLE design)
At the start: 137 parts

Commit message: added 18650 holder
Parts:
- added N1: BSS123, transistor-small-signal:BSS123
- added P1, P10, P11, P12, P2, P3, P4, P5, P6, P7, P8, P9: BSS84, transistor-small-signal:BSS84
Connections:
- new net BGND: BAT_TERMINALS.1, N1.S
- new net BT1: BAT_TERMINALS.2, P1.D
- new net BT10: BAT_TERMINALS.11
- new net BT11: BAT_TERMINALS.12
- new net BT12: BAT_TERMINALS.13
- new net BT2: BAT_TERMINALS.3
- new net BT3: BAT_TERMINALS.4
- new net BT4: BAT_TERMINALS.5
- new net BT5: BAT_TERMINALS.6
- new net BT6: BAT_TERMINALS.7
- new net BT7: BAT_TERMINALS.8
- new net BT8: BAT_TERMINALS.9
- new net BT9: BAT_TERMINALS.10
- new net N$47: P1.S, RBH1.2
- net 5V: now also N1.G
- net AGND: now also N1.D, P1.G; no longer BAT_TERMINALS.13
- net B1: no longer BAT_TERMINALS.12, RBH1.2
- net B10: no longer BAT_TERMINALS.3, RBH10.2
- net B11: no longer BAT_TERMINALS.2, RBH11.2
- net B12: no longer BAT_TERMINALS.1, RBH12.2
- net B2: no longer BAT_TERMINALS.11, RBH2.2
- net B3: no longer BAT_TERMINALS.10, RBH3.2
- net B4: no longer BAT_TERMINALS.9, RBH4.2
- net B5: no longer BAT_TERMINALS.8, RBH5.2
- net B6: no longer BAT_TERMINALS.7, RBH6.2
- net B7: no longer BAT_TERMINALS.6, RBH7.2
- net B8: no longer BAT_TERMINALS.5, RBH8.2
- net B9: no longer BAT_TERMINALS.4, RBH9.2
Other:
- moved on the sheet: C17, C18, C19, C20, C21, C22, C23, C24, R10, R11, R12, R13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
