File: projects/MotorDriver/TestV1.0.brd (EAGLE design)
At the start: 160 x 100 mm, 56 parts, among them IC1 7805TV, IC2 7812TV, J1 ARDUINO_UNO_R3, Q1 IRF9530, Q2 IRF9530, Q3 IRF9530, Q4 IRF9530, Q5 IRF9530, Q6 IRF9530

Commit message: added hall effect test board
Parts:
- removed IC1: 7805TV, linear:TO220V
- removed IC2: 7812TV, linear:TO220V
- removed U$4, U$5, U$6: WIRE_SOLDER_PAD, ISCTRainingProgram:SOLDER_PAD
- added MAX17604_B: MAX17604, st-microelectronics:SO08
- added R19, R20, R21: 0, eagle-ltspice:R0603
- renumbered U$1 to MAX17604_A, U$2 to MAX17604_C, U$3 to MAX17604_D
Connections:
- removed net N$3: Q1.D, Q2.S, R14.1, U$4.1
- removed net N$4: Q3.D, Q4.S, R16.2, U$5.1
- removed net N$5: Q5.D, Q6.S, R18.1, U$6.1
- new net A: Q1.D, Q2.S, R19.2
- new net A_MINOR: R14.1, R19.1
- new net B: Q3.D, Q4.S, R20.2
- new net B_MINOR: R16.2, R20.1
- new net C: Q5.D, Q6.S, R21.2
- new net C_MINOR: R18.1, R21.1
- new net N$30: X1.2
- new net N$36: R10.2, R11.2, R12.2, R7.1, R8.1, R9.2
- new net N$38: X1.1
- net HV+: no longer C1.+, C2.+, C3.+, IC1.1, IC2.1, X1.2
- net HV-: no longer C1.-, C2.-, C3.-, IC1.2, IC2.2, MAX17604_A.3, MAX17604_C.3, MAX17604_D.3, R10.2, R11.2, R12.2, R7.1, R8.1, R9.2, X1.1
- net HV12: no longer C4.1, IC2.3, MAX17604_A.6, MAX17604_C.6, MAX17604_D.6
- net HV5: no longer IC1.3
- net N$1: no longer MAX17604_A.7
- net N$10: no longer MAX17604_A.2
- net N$11: no longer MAX17604_A.4
- net N$12: no longer MAX17604_C.2
- net N$13: no longer MAX17604_C.4
- net N$14: no longer MAX17604_D.2
- net N$15: no longer MAX17604_D.4
- net N$2: no longer MAX17604_A.5
- net N$6: no longer MAX17604_C.7
- net N$7: no longer MAX17604_C.5
- net N$8: no longer MAX17604_D.7
- net N$9: no longer MAX17604_D.5
Routing:
- net HV12: track 214.8 -> 0.00 mm, vias 5 -> 0
- net N$5: track 127.5 -> 0.00 mm, vias 1 -> 0
- net N$18: track 123.5 -> 0.00 mm
- net AGND: track 109.0 -> 0.00 mm, vias 3 -> 0
- net N$4: track 108.8 -> 0.00 mm, vias 1 -> 0
- net 5V: track 103.3 -> 0.00 mm
- net N$3: track 97.2 -> 0.00 mm
- net HV-: track 76.6 -> 0.00 mm, vias 15 -> 0
- net A2: track 75.1 -> 0.00 mm, vias 1 -> 0
- net A1: track 73.0 -> 0.00 mm, vias 1 -> 0
- net A0: track 70.9 -> 0.00 mm, vias 1 -> 0
- net HV5: track 69.7 -> 0.00 mm, vias 2 -> 0
- net N$10: track 58.4 -> 0.00 mm, vias 1 -> 0
- net N$13: track 55.3 -> 0.00 mm
- net N$11: track 55.2 -> 0.00 mm, vias 2 -> 0
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